File: ESP_Programmer.sch (KiCad schematic (older format))
At the start: 26 parts, among them J1 USB_B_Micro, J2 Conn_01x04_Female, J3 FTDI_Header, J4 ESP_PROG, Q1 MBT3904DW1T1G, SW1 SW_SPST_SM_DP, SW2 SW_SPST_SM_DP, U1 FT232RL-REEL

Commit message: Added readme
Parts:
- J3: symbol avr-arduino:FTDI_Header -> ESP_Programmer-rescue:FTDI_Header-avr-arduino
- Q1: symbol dk_Transistors-Bipolar-BJT-Arrays:MBT3904DW1T1G -> ESP_Programmer-rescue:MBT3904DW1T1G-dk_Transistors-Bipolar-BJT-Arrays
- U1: symbol dk_Interface-Controllers:FT232RL-REEL -> ESP_Programmer-rescue:FT232RL-REEL-dk_Interface-Controllers
Changed lines of the file:
@@
 	8150 4050 8300 4050
 $Comp
-L dk_Interface-Controllers:FT232RL-REEL U1
+L ESP_Programmer-rescue:FT232RL-REEL-dk_Interface-Controllers U1
 U 1 1 611A732D
 P 7750 3750
@@
 Connection ~ 3950 4300
 $Comp
-L avr-arduino:FTDI_Header J3
+L ESP_Programmer-rescue:FTDI_Header-avr-arduino J3
 U 1 1 611F70B9
 P 5250 3800
@@
 	5450 4750 5450 4850
 $Comp
-L dk_Transistors-Bipolar-BJT-Arrays:MBT3904DW1T1G Q1
+L ESP_Programmer-rescue:MBT3904DW1T1G-dk_Transistors-Bipolar-BJT-Arrays Q1
 U 1 1 61214337
 P 6150 2750

Commit message: Add images
Parts:
- J1: symbol Connector:USB_B_Micro -> ESP_Programmer-rescue:USB_B_Micro-Connector
Changed lines of the file:
@@
 $EndDescr
 $Comp
-L Connector:USB_B_Micro J1
+L ESP_Programmer-rescue:USB_B_Micro-Connector J1
 U 1 1 611828BD
 P 3350 3050

Commit message: V2 led's and notes about C6 & C7
Parts:
- added R5, R6: 270R, symbol Device:R
- C6: value 10uF -> 10uF (optional)
- C7: value 0.1uF -> 0.1uF (optional)
Connections:
- net +5V: now also D1.2 (A), D2.2 (A)
- net GND: no longer D1.1 (K), D2.1 (K)
- net RXLED: now also R5.2; no longer D1.2 (A)
- net TXLED: now also R6.2; no longer D2.2 (A)
- new net: D1.1 (K), R5.1
- new net: D2.1 (K), R6.1
Other:
- note added: "Don't include these \non an ESP01 as they \nmess with I2C"
- moved on the sheet: D1, D2
Changed lines of the file:
@@
 Wire Wire Line
 	6900 4750 7050 4750
-Text GLabel 4050 4800 3    50   Input ~ 0
+Text GLabel 4350 5000 3    50   Input ~ 0
 TXLED
-Text GLabel 3900 4800 3    50   Input ~ 0
+Text GLabel 3900 5000 3    50   Input ~ 0
 RXLED
 $Comp
 L Device:LED D1
 U 1 1 611EC1D4
-P 3900 4550
-F 0 "D1" V 3800 4350 50  0000 L CNN
-F 1 "LED" V 3900 4350 50  0000 L CNN
-F 2 "LED_SMD:LED_1206_3216Metric_Pad1.42x1.75mm_HandSolder" H 3900 4550 50  0001 C CNN
-F 3 "~" H 3900 4550 50  0001 C CNN
-	1    3900 4550
-	0    1    1    0
+P 3900 4250
+F 0 "D1" V 3800 4050 50  0000 L CNN
+F 1 "LED" V 3900 4050 50  0000 L CNN
+F 2 "LED_SMD:LED_1206_3216Metric_Pad1.42x1.75mm_HandSolder" H 3900 4250 50  0001 C CNN
+F 3 "~" H 3900 4250 50  0001 C CNN
+	1    3900 4250
+	0    -1   -1   0
 $EndComp
 $Comp
 L Device:LED D2
 U 1 1 611EDE91
-P 4050 4550
-F 0 "D2" V 3950 4650 50  0000 L CNN
-F 1 "LED" V 4050 4650 50  0000 L CNN
-F 2 "LED_SMD:LED_1206_3216Metric_Pad1.42x1.75mm_HandSolder" H 4050 4550 50  0001 C CNN
-F 3 "~" H 4050 4550 50  0001 C CNN
-	1    4050 4550
-	0    1    1    0
-$EndComp
-Wire Wire Line
-	3900 4700 3900 4800
-Wire Wire Line
-	4050 4700 4050 4800
-$Comp
-L power:GND #PWR0111
-U 1 1 611F3DD3
-P 3950 4250
-F 0 "#PWR0111" H 3950 4000 50  0001 C CNN
-F 1 "GND" H 3955 4077 50  0000 C CNN
-F 2 "" H 3950 4250 50  0001 C CNN
-F 3 "" H 3950 4250 50  0001 C CNN
-	1    3950 4250
-	-1   0    0    1
-$EndComp
-Wire Wire Line
-	3900 4400 3900 4300
-Wire Wire Line
-	3900 4300 3950 4300
-Wire Wire Line
-	3950 4300 3950 4250
-Wire Wire Line
-	4050 4400 4050 4300
-Wire Wire Line
-	4050 4300 3950 4300
-Connection ~ 3950 4300
+P 4350 4250
+F 0 "D2" V 4250 4350 50  0000 L CNN
+F 1 "LED" V 4350 4350 50  0000 L CNN
+F 2 "LED_SMD:LED_1206_3216Metric_Pad1.42x1.75mm_HandSolder" H 4350 4250 50  0001 C CNN
+F 3 "~" H 4350 4250 50  0001 C CNN
+	1    4350 4250
+	0    -1   -1   0
+$EndComp
+Wire Wire Line
+	3900 4900 3900 5000
+Wire Wire Line
+	4350 4900 4350 5000
+Wire Wire Line
+	3900 4100 3900 4000
+Wire Wire Line
+	3900 4000 3950 4000
+Wire Wire Line
+	3950 4000 3950 3950
+Connection ~ 3950 4000
 $Comp
 L ESP_Programmer-rescue:FTDI_Header-avr-arduino J3
@@
 P 9950 1000
 F 0 "C6" H 10068 1046 50  0000 L CNN
-F 1 "10uF" H 10068 955 50  0000 L CNN
+F 1 "10uF (optional)" V 10250 700 50  0000 L CNN
 F 2 "Capacitor_Tantalum_SMD:CP_EIA-3216-18_Kemet-A_Pad1.58x1.35mm_HandSolder" H 9988 850 50  0001 C CNN
 F 3 "~" H 9950 1000 50  0001 C CNN
 	1    9950 1000
-	0    -1   -1   0
-$EndComp
-$Comp
-L Device:C C7
-U 1 1 6130A0A9
-P 9950 1300
-F 0 "C7" H 9750 1350 50  0000 L CNN
-F 1 "0.1uF" H 9650 1250 50  0000 L CNN
-F 2 "Capacitor_SMD:C_1206_3216Metric_Pad1.42x1.75mm_HandSolder" H 9988 1150 50  0001 C CNN
-F 3 "~" H 9950 1300 50  0001 C CNN
-	1    9950 1300
 	0    -1   -1   0
 $EndComp
@@
 Wire Wire Line
 	9350 1400 9350 1250
+$Comp
+L Device:C C7
+U 1 1 6130A0A9
+P 9950 1300
+F 0 "C7" H 9750 1350 50  0000 L CNN
+F 1 "0.1uF (optional)" V 9700 950 50  0000 L CNN
+F 2 "Capacitor_SMD:C_1206_3216Metric_Pad1.42x1.75mm_HandSolder" H 9988 1150 50  0001 C CNN
+F 3 "~" H 9950 1300 50  0001 C CNN
+	1    9950 1300
+	0    -1   -1   0
+$EndComp
+$Comp
+L power:+5V #PWR?
+U 1 1 627C4B07
+P 3950 3950
+F 0 "#PWR?" H 3950 3800 50  0001 C CNN
+F 1 "+5V" H 3965 4123 50  0000 C CNN
+F 2 "" H 3950 3950 50  0001 C CNN
+F 3 "" H 3950 3950 50  0001 C CNN
+	1    3950 3950
+	1    0    0    -1
+$EndComp
+Wire Wire Line
+	4350 4000 4350 4100
+Wire Wire Line
+	3950 4000 4350 4000
+$Comp
+L Device:R R6
+U 1 1 627E5AD6
+P 4350 4750
+F 0 "R6" H 4420 4796 50  0000 L CNN
+F 1 "270R" H 4420 4705 50  0000 L CNN
+F 2 "" V 4280 4750 50  0001 C CNN
+F 3 "~" H 4350 4750 50  0001 C CNN
+	1    4350 4750
+	1    0    0    -1
+$EndComp
+$Comp
+L Device:R R5
+U 1 1 627E6591
+P 3900 4750
+F 0 "R5" H 3970 4796 50  0000 L CNN
+F 1 "270R" H 3970 4705 50  0000 L CNN
+F 2 "" V 3830 4750 50  0001 C CNN
+F 3 "~" H 3900 4750 50  0001 C CNN
+	1    3900 4750
+	1    0    0    -1
+$EndComp
+Wire Wire Line
+	4350 4400 4350 4600
+Wire Wire Line
+	3900 4400 3900 4600
+Text Notes 10350 1050 0    50   ~ 0
+Don't include these \non an ESP01 as they \nmess with I2C
 $EndSCHEMATC
